File: 12f675-mppt.sch (KiCad schematic (older format))
At the start: 31 parts, among them IC1 PIC12F629-I/P, Q1 BUK9511-55A127, Q2 BUK9511-55A127, Q3 2N2222A, Q4 2N2222A, Q5 2N2907A, U1 7805, U2 LM358N

Commit message: Change Schematic. Use Reference voltage(pin 6). More Resistance on FET.
Parts:
- added D6: D, symbol D
- added D7, D8, D9: LED, symbol LED
- added R14: 4.7k, symbol R
- R1: value 10k -> 4.7k
Connections:
- net labels added: 2.5v, 3.6v
- wire segments 66 -> 76
Other:
- note added: "Max 25V"
- note removed: "Max 36V"
Changed lines of the file:
@@
 Sheet 1 1
 Title "Simple MPPT with 12F675"
-Date "2015-08-12"
-Rev "1.0b"
+Date "2015-08-13"
+Rev "1.1"
 Comp ""
 Comment1 ""
@@
 L Q_NMOS_GDS Q1
 U 1 1 55C339A5
-P 8300 5400
-F 0 "Q1" H 8600 5450 50  0000 R CNN
-F 1 "BUK9511-55A127" H 9200 5350 50  0000 R CNN
-F 2 "" H 8500 5500 29  0000 C CNN
-F 3 "" H 8300 5400 60  0000 C CNN
-	1    8300 5400
-	1    0    0    -1
+P 8500 5400
+F 0 "Q1" H 8800 5450 50  0000 R CNN
+F 1 "BUK9511-55A127" H 9400 5350 50  0000 R CNN
+F 2 "" H 8700 5500 29  0000 C CNN
+F 3 "" H 8500 5400 60  0000 C CNN
+	1    8500 5400
+	-1   0    0    -1
 $EndComp
 $Comp
@@
 L R R1
 U 1 1 55C344FE
-P 8100 5050
-F 0 "R1" V 8180 5050 50  0000 C CNN
-F 1 "10k" V 8100 5050 50  0000 C CNN
-F 2 "" V 8030 5050 30  0000 C CNN
-F 3 "" H 8100 5050 30  0000 C CNN
-	1    8100 5050
-	-1   0    0    1
+P 8650 4450
+F 0 "R1" V 8730 4450 50  0000 C CNN
+F 1 "4.7k" V 8650 4450 50  0000 C CNN
+F 2 "" V 8580 4450 30  0000 C CNN
+F 3 "" H 8650 4450 30  0000 C CNN
+	1    8650 4450
+	0    -1   -1   0
 $EndComp
 $Comp
@@
 	3050 3400 3850 3400
 Wire Wire Line
-	1600 5600 8400 5600
+	1600 5600 9050 5600
 Wire Wire Line
 	7400 5600 7400 5250
 Wire Wire Line
-	3500 4450 8100 4450
+	3500 4450 8500 4450
 Wire Wire Line
 	3500 2350 3500 4450
@@
 L R R8
 U 1 1 55C3B177
-P 5650 4200
-F 0 "R8" V 5730 4200 50  0000 C CNN
-F 1 "10k" V 5650 4200 50  0000 C CNN
-F 2 "" V 5580 4200 30  0000 C CNN
-F 3 "" H 5650 4200 30  0000 C CNN
-	1    5650 4200
+P 5450 4200
+F 0 "R8" V 5530 4200 50  0000 C CNN
+F 1 "10k" V 5450 4200 50  0000 C CNN
+F 2 "" V 5380 4200 30  0000 C CNN
+F 3 "" H 5450 4200 30  0000 C CNN
+	1    5450 4200
 	-1   0    0    1
 $EndComp
 Wire Wire Line
-	5650 4350 5650 4600
-Wire Wire Line
-	5650 4600 2100 4600
+	5450 4350 5450 4600
+Wire Wire Line
+	5450 4600 2100 4600
 Wire Wire Line
 	2100 4600 2100 3500
@@
 Connection ~ 1850 3500
 Wire Wire Line
-	5650 4050 5650 3800
-Wire Wire Line
-	5650 3800 5250 3800
+	5450 4050 5450 3800
+Wire Wire Line
+	5450 3800 5250 3800
 $Comp
 L R R6
@@
 Connection ~ 6600 2350
 Connection ~ 7400 5600
-Wire Wire Line
-	8100 4450 8100 4900
 Connection ~ 7400 4450
-Wire Wire Line
-	8100 5200 8100 5400
 Wire Wire Line
 	9500 2750 9500 2650
@@
 Connection ~ 8400 3950
 Text Notes 1400 3650 0    60   ~ 0
-Max 36V
+Max 25V
+$Comp
+L D D6
+U 1 1 55CC95CF
+P 9050 4600
+F 0 "D6" H 9050 4700 50  0000 C CNN
+F 1 "D" H 9050 4500 50  0000 C CNN
+F 2 "" H 9050 4600 60  0000 C CNN
+F 3 "" H 9050 4600 60  0000 C CNN
+	1    9050 4600
+	0    -1   -1   0
+$EndComp
+$Comp
+L LED D7
+U 1 1 55CC9696
+P 9050 5050
+F 0 "D7" H 9050 5150 50  0000 C CNN
+F 1 "LED" H 9050 4950 50  0000 C CNN
+F 2 "" H 9050 5050 60  0000 C CNN
+F 3 "" H 9050 5050 60  0000 C CNN
+	1    9050 5050
+	0    -1   -1   0
+$EndComp
+Wire Wire Line
+	9050 5600 9050 5250
+Connection ~ 8400 5600
+Wire Wire Line
+	9050 4850 9050 4750
+Wire Wire Line
+	8800 4450 9050 4450
+Wire Wire Line
+	8700 5400 8700 4750
+Wire Wire Line
+	8700 4750 8850 4750
+Wire Wire Line
+	8850 4750 8850 4450
+Connection ~ 8850 4450
+$Comp
+L LED D9
+U 1 1 55CCC105
+P 5650 5350
+F 0 "D9" H 5650 5450 50  0000 C CNN
+F 1 "LED" H 5650 5250 50  0000 C CNN
+F 2 "" H 5650 5350 60  0000 C CNN
+F 3 "" H 5650 5350 60  0000 C CNN
+	1    5650 5350
+	0    -1   -1   0
+$EndComp
+$Comp
+L LED D8
+U 1 1 55CCC217
+P 5650 4850
+F 0 "D8" H 5650 4950 50  0000 C CNN
+F 1 "LED" H 5650 4750 50  0000 C CNN
+F 2 "" H 5650 4850 60  0000 C CNN
+F 3 "" H 5650 4850 60  0000 C CNN
+	1    5650 4850
+	0    -1   -1   0
+$EndComp
+$Comp
+L R R14
+U 1 1 55CCC2B4
+P 5650 4200
+F 0 "R14" V 5730 4200 50  0000 C CNN
+F 1 "4.7k" V 5650 4200 50  0000 C CNN
+F 2 "" V 5580 4200 30  0000 C CNN
+F 3 "" H 5650 4200 30  0000 C CNN
+	1    5650 4200
+	1    0    0    -1
+$EndComp
+Wire Wire Line
+	5650 4350 5650 4650
+Wire Wire Line
+	5650 5050 5650 5150
+Wire Wire Line
+	5650 5550 5650 5600
+Connection ~ 5650 5600
+Wire Wire Line
+	5650 4050 5750 4050
+Wire Wire Line
+	5750 3500 5750 4450
+Connection ~ 5750 4450
+Wire Wire Line
+	5750 3500 5250 3500
+Connection ~ 5750 4050
+Text Label 8950 4450 0    60   ~ 0
+2.5v
+Text Label 5550 3500 0    60   ~ 0
+3.6v
 $EndSCHEMATC

Commit message: More working on current sensing. Add 1uF capacitor to schematic.
Parts:
- added C5: 1u, symbol CP
- C1: value 470uF -> 3300u
Connections:
- wire segments 76 -> 79
Changed lines of the file:
@@
 Sheet 1 1
 Title "Simple MPPT with 12F675"
-Date "2015-08-13"
-Rev "1.1"
+Date "2015-08-14"
+Rev "1.1a"
 Comp ""
 Comment1 ""
@@
 U 1 1 55C339A5
 P 8500 5400
-F 0 "Q1" H 8800 5450 50  0000 R CNN
-F 1 "BUK9511-55A127" H 9400 5350 50  0000 R CNN
+F 0 "Q1" H 8750 5300 50  0000 R CNN
+F 1 "BUK9511-55A127" H 8700 5100 50  0000 R CNN
 F 2 "" H 8700 5500 29  0000 C CNN
 F 3 "" H 8500 5400 60  0000 C CNN
@@
 P 9500 2500
 F 0 "C1" H 9525 2600 50  0000 L CNN
-F 1 "470uF" H 9525 2400 50  0000 L CNN
+F 1 "3300u" H 9525 2400 50  0000 L CNN
 F 2 "" H 9538 2350 30  0000 C CNN
 F 3 "" H 9500 2500 60  0000 C CNN
@@
 Text Label 5550 3500 0    60   ~ 0
 3.6v
+$Comp
+L CP C5
+U 1 1 55CDDBD9
+P 8050 5150
+F 0 "C5" H 8075 5250 50  0000 L CNN
+F 1 "1u" H 8075 5050 50  0000 L CNN
+F 2 "" H 8088 5000 30  0000 C CNN
+F 3 "" H 8050 5150 60  0000 C CNN
+	1    8050 5150
+	1    0    0    -1
+$EndComp
+Wire Wire Line
+	8050 5300 8050 5600
+Connection ~ 8050 5600
+Wire Wire Line
+	8050 5000 8050 4900
+Wire Wire Line
+	8050 4900 8400 4900
+Connection ~ 8400 4900
 $EndSCHEMATC

Commit message: Correct current sensing.
Parts:
- C5: value 1u -> 2.2u(or higher)
Connections:
- wire segments 79 -> 78
Changed lines of the file:
@@
 Sheet 1 1
 Title "Simple MPPT with 12F675"
-Date "2015-08-14"
-Rev "1.1a"
+Date "2015-08-15"
+Rev "1.1b"
 Comp ""
 Comment1 ""
@@
 Heat Sink
 Wire Notes Line
-	6450 3750 9400 3750
+	9400 5850 9400 3750
 Wire Notes Line
-	9400 3750 9400 5850
-Wire Notes Line
-	9400 5850 6450 5850
-Wire Notes Line
-	6450 5850 6450 3750
+	5900 5850 9400 5850
 $Comp
 L R R11
@@
 L CP C5
 U 1 1 55CDDBD9
-P 8050 5150
-F 0 "C5" H 8075 5250 50  0000 L CNN
-F 1 "1u" H 8075 5050 50  0000 L CNN
-F 2 "" H 8088 5000 30  0000 C CNN
-F 3 "" H 8050 5150 60  0000 C CNN
-	1    8050 5150
-	1    0    0    -1
-$EndComp
-Wire Wire Line
-	8050 5300 8050 5600
-Connection ~ 8050 5600
-Wire Wire Line
-	8050 5000 8050 4900
-Wire Wire Line
-	8050 4900 8400 4900
-Connection ~ 8400 4900
+P 6000 4900
+F 0 "C5" H 6025 5000 50  0000 L CNN
+F 1 "2.2u(or higher)" H 6025 4800 50  0000 L CNN
+F 2 "" H 6038 4750 30  0000 C CNN
+F 3 "" H 6000 4900 60  0000 C CNN
+	1    6000 4900
+	1    0    0    -1
+$EndComp
+Wire Wire Line
+	6000 5050 6000 5600
+Connection ~ 6000 5600
+Wire Wire Line
+	6000 4750 6000 3600
+Connection ~ 6000 3600
+Wire Notes Line
+	5900 3500 5900 5850
+Wire Notes Line
+	5900 3500 6450 3500
+Wire Notes Line
+	6450 3500 6450 3750
+Wire Notes Line
+	6450 3750 9400 3750
 $EndSCHEMATC

Commit message: Fix circuit and code changes.
Parts:
- added C6: 2.2u(or higher), symbol CP
- C3: value 10u -> 100u
Connections:
- wire segments 78 -> 85
Changed lines of the file:
@@
 Sheet 1 1
 Title "Simple MPPT with 12F675"
-Date "2015-08-15"
-Rev "1.1b"
+Date "2015-08-16"
+Rev "1.1c"
 Comp ""
 Comment1 ""
@@
 	7400 5600 7400 5250
 Wire Wire Line
-	3500 4450 8500 4450
-Wire Wire Line
-	3500 2350 3500 4450
+	3500 2350 3500 6100
 Connection ~ 3500 3400
 Wire Wire Line
@@
 L R R8
 U 1 1 55C3B177
-P 5450 4200
-F 0 "R8" V 5530 4200 50  0000 C CNN
-F 1 "10k" V 5450 4200 50  0000 C CNN
-F 2 "" V 5380 4200 30  0000 C CNN
-F 3 "" H 5450 4200 30  0000 C CNN
-	1    5450 4200
-	-1   0    0    1
-$EndComp
-Wire Wire Line
-	5450 4350 5450 4600
-Wire Wire Line
-	5450 4600 2100 4600
-Wire Wire Line
-	2100 4600 2100 3500
+P 4550 4400
+F 0 "R8" V 4630 4400 50  0000 C CNN
+F 1 "10k" V 4550 4400 50  0000 C CNN
+F 2 "" V 4480 4400 30  0000 C CNN
+F 3 "" H 4550 4400 30  0000 C CNN
+	1    4550 4400
+	0    -1   -1   0
+$EndComp
 Wire Wire Line
 	2100 3500 1850 3500
 Connection ~ 1850 3500
-Wire Wire Line
-	5450 4050 5450 3800
-Wire Wire Line
-	5450 3800 5250 3800
 $Comp
 L R R6
 U 1 1 55C3BCB8
-P 5250 4900
-F 0 "R6" V 5330 4900 50  0000 C CNN
-F 1 "1k" V 5250 4900 50  0000 C CNN
-F 2 "" V 5180 4900 30  0000 C CNN
-F 3 "" H 5250 4900 30  0000 C CNN
-	1    5250 4900
+P 4900 4900
+F 0 "R6" V 4980 4900 50  0000 C CNN
+F 1 "1k" V 4900 4900 50  0000 C CNN
+F 2 "" V 4830 4900 30  0000 C CNN
+F 3 "" H 4900 4900 30  0000 C CNN
+	1    4900 4900
 	-1   0    0    1
 $EndComp
@@
 L LED D4
 U 1 1 55C3BFD1
-P 5250 5350
-F 0 "D4" H 5250 5450 50  0000 C CNN
-F 1 "LED" H 5250 5250 50  0000 C CNN
-F 2 "" H 5250 5350 60  0000 C CNN
-F 3 "" H 5250 5350 60  0000 C CNN
-	1    5250 5350
-	0    -1   -1   0
-$EndComp
-Wire Wire Line
-	5250 5550 5250 5600
-Connection ~ 5250 5600
-Wire Wire Line
-	5250 5150 5250 5050
-Wire Wire Line
-	5250 3900 5250 4750
+P 4900 5350
+F 0 "D4" H 4900 5450 50  0000 C CNN
+F 1 "LED" H 4900 5250 50  0000 C CNN
+F 2 "" H 4900 5350 60  0000 C CNN
+F 3 "" H 4900 5350 60  0000 C CNN
+	1    4900 5350
+	0    -1   -1   0
+$EndComp
+Wire Wire Line
+	4900 5550 4900 5600
+Connection ~ 4900 5600
+Wire Wire Line
+	4900 5150 4900 5050
 $Comp
 L D D5
@@
 P 3100 3700
 F 0 "C3" H 3125 3800 50  0000 L CNN
-F 1 "10u" H 3125 3600 50  0000 L CNN
+F 1 "100u" H 3125 3600 50  0000 L CNN
 F 2 "" H 3138 3550 30  0000 C CNN
 F 3 "" H 3100 3700 60  0000 C CNN
@@
 Text Label 7050 3600 2    60   ~ 0
 PV-Current
-Text Label 4250 4600 2    60   ~ 0
+Text Label 4200 4400 2    60   ~ 0
 PV-Voltage
 Text Notes 8900 5200 2    60   ~ 0
@@
 L R R11
 U 1 1 55C4C21C
-P 6200 3600
-F 0 "R11" V 6280 3600 50  0000 C CNN
-F 1 "10k" V 6200 3600 50  0000 C CNN
-F 2 "" V 6130 3600 30  0000 C CNN
-F 3 "" H 6200 3600 30  0000 C CNN
-	1    6200 3600
+P 6400 3600
+F 0 "R11" V 6480 3600 50  0000 C CNN
+F 1 "10k" V 6400 3600 50  0000 C CNN
+F 2 "" V 6330 3600 30  0000 C CNN
+F 3 "" H 6400 3600 30  0000 C CNN
+	1    6400 3600
 	0    1    1    0
 $EndComp
 Wire Wire Line
-	6350 3600 8000 3600
-Wire Wire Line
-	6050 3600 5250 3600
+	6550 3600 8000 3600
+Wire Wire Line
+	5250 3600 6250 3600
 $Comp
 L R R12
@@
 	8800 4450 9050 4450
 Wire Wire Line
-	8700 5400 8700 4750
-Wire Wire Line
-	8700 4750 8850 4750
-Wire Wire Line
-	8850 4750 8850 4450
+	8850 4450 8850 5400
 Connection ~ 8850 4450
 $Comp
@@
 Connection ~ 5650 5600
 Wire Wire Line
-	5650 4050 5750 4050
-Wire Wire Line
-	5750 3500 5750 4450
-Connection ~ 5750 4450
-Wire Wire Line
-	5750 3500 5250 3500
-Connection ~ 5750 4050
+	5650 4050 6000 4050
 Text Label 8950 4450 0    60   ~ 0
 2.5v
-Text Label 5550 3500 0    60   ~ 0
+Text Label 5350 3500 0    60   ~ 0
 3.6v
 $Comp
 L CP C5
 U 1 1 55CDDBD9
-P 6000 4900
-F 0 "C5" H 6025 5000 50  0000 L CNN
-F 1 "2.2u(or higher)" H 6025 4800 50  0000 L CNN
-F 2 "" H 6038 4750 30  0000 C CNN
-F 3 "" H 6000 4900 60  0000 C CNN
-	1    6000 4900
-	1    0    0    -1
-$EndComp
-Wire Wire Line
-	6000 5050 6000 5600
-Connection ~ 6000 5600
-Wire Wire Line
-	6000 4750 6000 3600
-Connection ~ 6000 3600
+P 6100 4900
+F 0 "C5" H 6125 5000 50  0000 L CNN
+F 1 "2.2u(or higher)" H 6125 4800 50  0000 L CNN
+F 2 "" H 6138 4750 30  0000 C CNN
+F 3 "" H 6100 4900 60  0000 C CNN
+	1    6100 4900
+	1    0    0    -1
+$EndComp
+Wire Wire Line
+	6100 5050 6100 5600
+Connection ~ 6100 5600
+Wire Wire Line
+	6100 4750 6100 3600
+Connection ~ 6100 3600
 Wire Notes Line
 	5900 3500 5900 5850
 Wire Notes Line
-	5900 3500 6450 3500
+	5900 3500 6500 3500
 Wire Notes Line
-	6450 3500 6450 3750
+	6500 3500 6700 3750
 Wire Notes Line
-	6450 3750 9400 3750
+	6700 3750 9400 3750
+$Comp
+L CP C6
+U 1 1 55D02AF9
+P 5200 5150
+F 0 "C6" H 5100 5400 50  0000 L CNN
+F 1 "2.2u(or higher)" H 5000 5300 50  0000 L CNN
+F 2 "" H 5238 5000 30  0000 C CNN
+F 3 "" H 5200 5150 60  0000 C CNN
+	1    5200 5150
+	1    0    0    -1
+$EndComp
+Wire Wire Line
+	3500 6100 8150 6100
+Wire Wire Line
+	8150 4450 8150 6100
+Wire Wire Line
+	5250 3900 5250 4300
+Wire Wire Line
+	5250 4300 4900 4300
+Wire Wire Line
+	4900 4300 4900 4750
+Wire Wire Line
+	5200 5300 5200 5600
+Connection ~ 5200 5600
+Wire Wire Line
+	2100 3500 2100 4400
+Wire Wire Line
+	2100 4400 4400 4400
+Wire Wire Line
+	4700 4400 5400 4400
+Wire Wire Line
+	5400 4400 5400 3800
+Wire Wire Line
+	5400 3800 5250 3800
+Wire Wire Line
+	5200 5000 5200 4400
+Connection ~ 5200 4400
+Connection ~ 8150 4450
+Wire Wire Line
+	5650 4500 5500 4500
+Wire Wire Line
+	5500 4500 5500 3500
+Connection ~ 5650 4500
+Wire Wire Line
+	6000 4450 8500 4450
+Wire Wire Line
+	6000 4050 6000 4450
+Wire Wire Line
+	5500 3500 5250 3500
+Wire Wire Line
+	8850 5400 8700 5400
 $EndSCHEMATC

Commit message: Simple is the best. replace loop code for maximum power calibration. Change 100k to 200k ohm because current sensing voltage is too low.
Parts:
- R2, R4: value 100k -> 200k
Changed lines of the file:
@@
 Sheet 1 1
 Title "Simple MPPT with 12F675"
-Date "2015-08-16"
-Rev "1.1c"
+Date "2015-08-18"
+Rev "1.1d"
 Comp ""
 Comment1 ""
@@
 P 7050 4250
 F 0 "R4" V 7130 4250 50  0000 C CNN
-F 1 "100k" V 7050 4250 50  0000 C CNN
+F 1 "200k" V 7050 4250 50  0000 C CNN
 F 2 "" V 6980 4250 30  0000 C CNN
 F 3 "" H 7050 4250 30  0000 C CNN
@@
 P 6700 5300
 F 0 "R2" V 6780 5300 50  0000 C CNN
-F 1 "100k" V 6700 5300 50  0000 C CNN
+F 1 "200k" V 6700 5300 50  0000 C CNN
 F 2 "" V 6630 5300 30  0000 C CNN
 F 3 "" H 6700 5300 30  0000 C CNN

Commit message: Change low pass filter at ADC inputs. Narrows voltage range at solar panel.
Parts:
- C1: value 3300u -> 100u
- C5, C6: value 2.2u(or higher) -> 10u
Changed lines of the file:
@@
 Sheet 1 1
 Title "Simple MPPT with 12F675"
-Date "2015-08-18"
-Rev "1.1d"
+Date "2015-08-22"
+Rev "1.1e"
 Comp ""
 Comment1 ""
@@
 P 9500 2500
 F 0 "C1" H 9525 2600 50  0000 L CNN
-F 1 "3300u" H 9525 2400 50  0000 L CNN
+F 1 "100u" H 9525 2400 50  0000 L CNN
 F 2 "" H 9538 2350 30  0000 C CNN
 F 3 "" H 9500 2500 60  0000 C CNN
@@
 P 6100 4900
 F 0 "C5" H 6125 5000 50  0000 L CNN
-F 1 "2.2u(or higher)" H 6125 4800 50  0000 L CNN
+F 1 "10u" H 6125 4800 50  0000 L CNN
 F 2 "" H 6138 4750 30  0000 C CNN
 F 3 "" H 6100 4900 60  0000 C CNN
@@
 P 5200 5150
 F 0 "C6" H 5100 5400 50  0000 L CNN
-F 1 "2.2u(or higher)" H 5000 5300 50  0000 L CNN
+F 1 "10u" H 5000 5300 50  0000 L CNN
 F 2 "" H 5238 5000 30  0000 C CNN
 F 3 "" H 5200 5150 60  0000 C CNN

Commit message: Reduce circuit parts. 3,6v to current sensing FET(low value on datasheet is 3v).
Parts:
- removed D6: D, symbol D
- removed D7: LED, symbol LED
- removed R1: 4.7k, symbol R
Connections:
- net labels removed: 2.5v
- wire segments 85 -> 83
Changed lines of the file:
@@
 Sheet 1 1
 Title "Simple MPPT with 12F675"
-Date "2015-08-22"
-Rev "1.1e"
+Date "2015-08-26"
+Rev "1.1f"
 Comp ""
 Comment1 ""
@@
 $EndComp
 $Comp
-L R R1
-U 1 1 55C344FE
-P 8650 4450
-F 0 "R1" V 8730 4450 50  0000 C CNN
-F 1 "4.7k" V 8650 4450 50  0000 C CNN
-F 2 "" V 8580 4450 30  0000 C CNN
-F 3 "" H 8650 4450 30  0000 C CNN
-	1    8650 4450
-	0    -1   -1   0
-$EndComp
-$Comp
 L LM358N U2
 U 2 1 55C3383E
@@
 Wire Wire Line
 	3050 3400 3850 3400
-Wire Wire Line
-	1600 5600 9050 5600
 Wire Wire Line
 	7400 5600 7400 5250
@@
 Max 25V
 $Comp
-L D D6
-U 1 1 55CC95CF
-P 9050 4600
-F 0 "D6" H 9050 4700 50  0000 C CNN
-F 1 "D" H 9050 4500 50  0000 C CNN
-F 2 "" H 9050 4600 60  0000 C CNN
-F 3 "" H 9050 4600 60  0000 C CNN
-	1    9050 4600
-	0    -1   -1   0
-$EndComp
-$Comp
-L LED D7
-U 1 1 55CC9696
-P 9050 5050
-F 0 "D7" H 9050 5150 50  0000 C CNN
-F 1 "LED" H 9050 4950 50  0000 C CNN
-F 2 "" H 9050 5050 60  0000 C CNN
-F 3 "" H 9050 5050 60  0000 C CNN
-	1    9050 5050
-	0    -1   -1   0
-$EndComp
-Wire Wire Line
-	9050 5600 9050 5250
-Connection ~ 8400 5600
-Wire Wire Line
-	9050 4850 9050 4750
-Wire Wire Line
-	8800 4450 9050 4450
-Wire Wire Line
-	8850 4450 8850 5400
-Connection ~ 8850 4450
-$Comp
 L LED D9
 U 1 1 55CCC105
@@
 Wire Wire Line
 	5650 4050 6000 4050
-Text Label 8950 4450 0    60   ~ 0
-2.5v
 Text Label 5350 3500 0    60   ~ 0
 3.6v
@@
 	3500 6100 8150 6100
 Wire Wire Line
-	8150 4450 8150 6100
+	8150 6100 8150 4450
 Wire Wire Line
 	5250 3900 5250 4300
@@
 	5200 5000 5200 4400
 Connection ~ 5200 4400
-Connection ~ 8150 4450
 Wire Wire Line
 	5650 4500 5500 4500
 Wire Wire Line
-	5500 4500 5500 3500
+	5500 3500 5500 6000
 Connection ~ 5650 4500
 Wire Wire Line
-	6000 4450 8500 4450
-Wire Wire Line
 	6000 4050 6000 4450
 Wire Wire Line
@@
 Wire Wire Line
 	8850 5400 8700 5400
+Wire Wire Line
+	5500 6000 8850 6000
+Wire Wire Line
+	8850 6000 8850 5400
+Connection ~ 5500 4500
+Wire Wire Line
+	6000 4450 8150 4450
+Wire Wire Line
+	1600 5600 8400 5600
+Text Label 8550 6000 0    60   ~ 0
+3.6v
 $EndSCHEMATC

Commit message: Change ADC low pass filter's resisters(10k to 100k). New code.
Parts:
- R11, R8: value 10k -> 100k
- R2, R4: value 200k -> 300k
Changed lines of the file:
@@
 Sheet 1 1
 Title "Simple MPPT with 12F675"
-Date "2015-08-26"
-Rev "1.1f"
+Date "2015-08-30"
+Rev "1.1h"
 Comp ""
 Comment1 ""
@@
 P 7050 4250
 F 0 "R4" V 7130 4250 50  0000 C CNN
-F 1 "200k" V 7050 4250 50  0000 C CNN
+F 1 "300k" V 7050 4250 50  0000 C CNN
 F 2 "" V 6980 4250 30  0000 C CNN
 F 3 "" H 7050 4250 30  0000 C CNN
@@
 P 4550 4400
 F 0 "R8" V 4630 4400 50  0000 C CNN
-F 1 "10k" V 4550 4400 50  0000 C CNN
+F 1 "100k" V 4550 4400 50  0000 C CNN
 F 2 "" V 4480 4400 30  0000 C CNN
 F 3 "" H 4550 4400 30  0000 C CNN
@@
 P 6400 3600
 F 0 "R11" V 6480 3600 50  0000 C CNN
-F 1 "10k" V 6400 3600 50  0000 C CNN
+F 1 "100k" V 6400 3600 50  0000 C CNN
 F 2 "" V 6330 3600 30  0000 C CNN
 F 3 "" H 6400 3600 30  0000 C CNN
@@
 P 6700 5300
 F 0 "R2" V 6780 5300 50  0000 C CNN
-F 1 "200k" V 6700 5300 50  0000 C CNN
+F 1 "300k" V 6700 5300 50  0000 C CNN
 F 2 "" V 6630 5300 30  0000 C CNN
 F 3 "" H 6700 5300 30  0000 C CNN
